Commit message: 3条蛇臂已生成，x轴装配尺寸还有些问题

File: src/raphael_robot_description/urdf/common/snake/snake_params.xacro (robot description, xacro)
@@ -1,8 +1,7 @@
-<?xml version="1.0"?>
+<?xml version="1.0" encoding="UTF-8"?>
 <!-- 蛇臂14节连杆参数：质量、半径、长度分块分组存放 -->
 <robot xmlns:xacro="http://www.ros.org/wiki/xacro">
     <xacro:property name="mesh_scale" value="0.001 0.001 0.001"/>
-    <xacro:property name="stl_path" value="package://raphael_robot_description/meshes/stl"/>
-    <xacro:property name="links_material" value="cold_blue_metal"/>
+    <xacro:property name="stl_path" value="package://raphael_robot_description/meshes/snake"/>
     <!-- ====================== 各连杆质量 m(kg) ====================== -->
     <xacro:property name="link0_m" value="0.10"/>

File: src/raphael_robot_description/urdf/raphael_robot.urdf.xacro (robot description, xacro)
@@ -1,11 +1,9 @@
 <?xml version="1.0"?>
 <robot name="raphael_robot" xmlns:xacro="http://www.ros.org/wiki/xacro">
-    <!-- 1 material + inertia -->
-    <xacro:include filename="$(find raphael_robot_description)/urdf/common/materials_inertia.xacro"/>
-    <!-- 2 params -->
-    <xacro:include filename="$(find raphael_robot_description)/urdf/common/robot_params.xacro"/>
-    <!-- 3 links -->
-    <xacro:include filename="$(find raphael_robot_description)/urdf/macros/robot_links.xacro"/>
-    <!-- 4 joints -->
-    <xacro:include filename="$(find raphael_robot_description)/urdf/macros/robot_joints.xacro"/>
+    <!-- 加载通用 material -->
+    <xacro:include filename="$(find raphael_robot_description)/urdf/common/materials.xacro"/>
+    <!-- 加载通用 inertia -->
+    <xacro:include filename="$(find raphael_robot_description)/urdf/common/inertia.xacro"/>
+    <!-- 加载总装模型 -->
+    <xacro:include filename="$(find raphael_robot_description)/urdf/assemble/global_mount.xacro"/>
 </robot>
